File: term/term.kicad_pcb (KiCad board)
At the start: 2 copper layers, 0 parts

Commit message: Add kicad project with stm32 module
Parts:
- added BT1: Battery, Battery:BatteryHolder_ComfortableElectronic_CH273-2450_1x2450, B.Cu at (154.7, 40.0)
- added C1: 100n, Capacitor_SMD:C_0805_2012Metric, B.Cu at (163.3, 67.1)
- added C10: 100n, Capacitor_SMD:C_0805_2012Metric, B.Cu at (159.3, 77.9)
- added C11: 22p, Capacitor_SMD:C_0805_2012Metric, B.Cu at (185.5, 52.8)
- added C2: 100n, Capacitor_SMD:C_0805_2012Metric, B.Cu at (174.7, 61.7)
- added C3: 100n, Capacitor_SMD:C_0805_2012Metric, B.Cu at (210.1, 27.2)
- added C4: 100n, Capacitor_SMD:C_0805_2012Metric, B.Cu at (163.3, 70.1)
- added C5: 100n, Capacitor_SMD:C_0805_2012Metric, B.Cu at (174.7, 58.7)
- added C6: 100n, Capacitor_SMD:C_0805_2012Metric, B.Cu at (206.8, 45.5)
- added C7: 100n, Capacitor_SMD:C_0805_2012Metric, B.Cu at (174.7, 55.8)
- added C8: 100n, Capacitor_SMD:C_0805_2012Metric, B.Cu at (154.9, 77.9)
- added C9: 22p, Capacitor_SMD:C_0805_2012Metric, B.Cu at (167.8, 67.1)
- added J4: Conn_ARM_JTAG_SWD_10, Connector_IDC:IDC-Header_2x05_P2.54mm_Vertical, B.Cu at (187.5, 31.9)
- added R1: 1k, Resistor_SMD:R_0805_2012Metric, B.Cu at (179.1, 55.8)
- added R2: 4k7, Resistor_SMD:R_0805_2012Metric, B.Cu at (167.8, 70.1)
- added R3: 10, Resistor_SMD:R_1210_3225Metric, B.Cu at (155.5, 74.3)
- added R4: 100k, Resistor_SMD:R_0805_2012Metric, B.Cu at (179.1, 58.7)
- added R5: 100k, Resistor_SMD:R_0805_2012Metric, B.Cu at (198.4, 44.7)
- added R6: 4k7, Resistor_SMD:R_0805_2012Metric, B.Cu at (190.5, 49.4)
- added R7: 4k7, Resistor_SMD:R_0805_2012Metric, B.Cu at (172.2, 67.1)
- added RV1: 10k, Potentiometer_THT:Potentiometer_ACP_CA9-V10_Vertical, B.Cu at (195.9, 33.9)
- added U1: 74HC595, Package_SO:SOIC-16_3.9x9.9mm_P1.27mm, B.Cu at (167.0, 87.7)
- added U2: WG12864A, Connector_PinHeader_2.54mm:PinHeader_1x20_P2.54mm_Vertical, F.Cu at (189.2, 101.6)
- added U3: STM32F103C8Tx, Package_QFP:LQFP-48_7x7mm_P0.5mm, B.Cu at (166.8, 60.0)
- added U4: FM24C64B, Package_SO:SOIC-8_3.9x4.9mm_P1.27mm, B.Cu at (156.9, 69.0)
- added Y1: 8MHz, Crystal:Resonator_SMD_muRata_CSTxExxV-3Pin_3.0x1.1mm, B.Cu at (160.9, 74.0)
- added Y2: 32678, Crystal:Crystal_SMD_3215-2Pin_3.2x1.5mm, B.Cu at (185.8, 49.6)
Routing:
- net GND: track 0.00 -> 24.7 mm
- net Net-(U1-Pad15): track 0.00 -> 19.1 mm
- net Net-(U1-Pad7): track 0.00 -> 14.6 mm
- net Net-(U1-Pad6): track 0.00 -> 14.1 mm
- net Net-(U1-Pad5): track 0.00 -> 13.5 mm
- net Net-(U1-Pad4): track 0.00 -> 13.0 mm
- net Net-(U1-Pad3): track 0.00 -> 12.5 mm
- net Net-(U1-Pad2): track 0.00 -> 12.0 mm
- net Net-(U1-Pad1): track 0.00 -> 11.4 mm
